File: COCHE_COMPETENCIA.kicad_sch (KiCad schematic)
At the start: 25 parts, among them J1 BAT, J2 SENSORES, J3 M1, J4 M2, SW1 SW_Push, SW2 SW_Push, U1 L7805, U2 ESP32-DEVKIT-V1, U3 DRV8833, U4 DRV8833

Commit message: V1 - MotorBoard 2025
Parts:
- removed J2: SENSORES, Connector_PinHeader_2.54mm:PinHeader_1x10_P2.54mm_Vertical, symbol Connector:Conn_01x10_Pin
- removed R4, R7: 0, Resistor_SMD:R_1206_3216Metric_Pad1.30x1.75mm_HandSolder, symbol Device:R
- added J2: SWITCH, Connector_PinHeader_2.54mm:PinHeader_1x03_P2.54mm_Vertical, symbol Connector:Conn_01x03_Pin
- added J6: SENSORES, Connector_PinHeader_2.54mm:PinHeader_1x11_P2.54mm_Vertical, symbol Connector:Conn_01x11_Pin
- added R1, R5: 0, Resistor_SMD:R_1206_3216Metric_Pad1.30x1.75mm_HandSolder, symbol Device:R
- renumbered J3 to J4, J4 to J5, R1 to R2, R2 to R3, R3 to R4, R5 to R7
Connections:
- net +3.3V: now also SW1.1, SW2.1, J6.1 (Pin_1)
- net BUZZER: now also U2.7 (TX2); no longer U2.5 (D4)
- net GND: now also D1.1 (K), J6.11 (Pin_11), R1.1, R1.2; no longer R4.2
- net IN_M1_A: now also U2.24 (D26), R5.1; no longer U2.20 (D35), U3.5 (IN2)
- net IN_M1_B: now also U2.23 (D25), U3.2 (IN3); no longer U2.21 (D32)
- net IN_M2_A: now also U2.11 (D21), U4.5 (IN2); no longer R6.1, U2.10 (D19)
- net IN_M2_B: now also R6.1, U2.9 (D18); no longer U2.11 (D21), U4.2 (IN3)
- net LED_LARGADA: now also R4.1, U2.28 (D13); no longer D1.2 (A), U2.19 (D34)
- net S1: now also U2.26 (D14), J6.9 (Pin_9); no longer U2.28 (D13)
- net S2: now also U2.25 (D27), J6.8 (Pin_8); no longer U2.27 (D12)
- net S3: now also U2.22 (D33), J6.7 (Pin_7); no longer U2.26 (D14)
- net S4: now also U2.21 (D32), J6.6 (Pin_6); no longer U2.25 (D27)
- net S5: now also U2.20 (D35), J6.5 (Pin_5); no longer U2.24 (D26)
- net S6: now also U2.19 (D34), J6.4 (Pin_4); no longer U2.23 (D25)
- net S7: now also U2.18 (VN), J6.3 (Pin_3); no longer U2.4 (D2)
- net S8: now also U2.17 (VP), J6.2 (Pin_2); no longer U2.3 (D15)
- net SLEEP_M1: now also U2.6 (RX2); no longer U2.22 (D33)
- net SLEEP_M2: now also U2.15 (D23); no longer U2.9 (D18)
- net SW1: now also U2.14 (D22); no longer U2.15 (D23)
- net SW2: now also U2.10 (D19); no longer U2.14 (D22)
- net VCC: now also J2.3 (Pin_3); no longer J1.1 (Pin_1)
- net +5V: now reaches C2.1, U1.3 (OUT), U2.30 (VIN)
- net at R6.2: now also U4.2 (IN3); no longer U4.5 (IN2)
- new net: D1.2 (A), R4.2
- new net: R5.2, U3.5 (IN2)
- new net: J1.1 (Pin_1), J2.1 (Pin_1), J2.2 (Pin_2)
- no-connect marks 0 -> 12
Other:
- moved on the sheet: BZ1, C1, C2, D1, J1, R2, R3, R4, R7, SW1, SW2, U1
