File: MATRIZ_COCHE_COMPETENCIA.kicad_pcb (KiCad board)
At the start: 2 copper layers, 238 x 198.6 mm, 174 parts, among them J1 BAT, J10 SENSORES, J11 BAT, J12 SWITCH, J13 M1, J14 M2, J15 SENSORES, J16 BAT, J17 SWITCH, J18 M1, J19 M2, J2 SWITCH, J20 SENSORES, J21 BAT, J22 SWITCH, J23 M1, J24 M2, J25 SENSORES, J26 BAT, J27 SWITCH, J28 M1, J29 M2, J3 BAT, J30 SENSORES, J4 M1, J5 M2, J6 SENSORES, J7 SWITCH, J8 M1, J9 M2, SW1 SW_Push, SW10 SW_Push, SW11 SW_Push, SW12 SW_Push, SW2 SW_Push, SW3 SW_Push, SW4 SW_Push, SW5 SW_Push, SW6 SW_Push, SW7 SW_Push, SW8 SW_Push, SW9 SW_Push, U1 L7805, U10 ESP32-DEVKIT-V1, U11 DRV8833, U12 DRV8833, U13 L7805, U14 ESP32-DEVKIT-V1, U15 DRV8833, U16 DRV8833, U17 L7805, U18 ESP32-DEVKIT-V1, U19 DRV8833, U2 ESP32-DEVKIT-V1, U20 DRV8833, U21 L7805, U22 ESP32-DEVKIT-V1, U23 DRV8833, U24 DRV8833, U3 DRV8833, U4 DRV8833, U5 L7805, U6 ESP32-DEVKIT-V1, U7 DRV8833, U8 DRV8833, U9 L7805

Commit message: V1 - Diagrama Draw.io y Mejoras documentacion
Parts:
- removed BZ1: Buzzer, Buzzer_Beeper:MagneticBuzzer_ProSignal_ABI-009-RC
- removed C1: 0.33u, Capacitor_SMD:C_1206_3216Metric_Pad1.33x1.80mm_HandSolder
- removed C2: 0.1u, Capacitor_SMD:C_1206_3216Metric_Pad1.33x1.80mm_HandSolder
- removed D1: LED_RED, LED_SMD:LED_1206_3216Metric_Pad1.42x1.75mm_HandSolder
- removed G*** (x3): LOGO, LOGO
- removed H1, H2, H3, H4: MountingHole, MountingHole:MountingHole_3mm
- removed J1: BAT, TerminalBlock_Phoenix:TerminalBlock_Phoenix_MKDS-1,5-2_1x02_P5.00mm_Horizontal
- removed J2: SWITCH, Connector_PinHeader_2.54mm:PinHeader_1x03_P2.54mm_Vertical
- removed R1, R5, R6, R7: 0, Resistor_SMD:R_1206_3216Metric_Pad1.30x1.75mm_HandSolder
- removed R2, R3: 10k, Resistor_SMD:R_1206_3216Metric_Pad1.30x1.75mm_HandSolder
- removed R4: 220, Resistor_SMD:R_1206_3216Metric_Pad1.30x1.75mm_HandSolder
- removed SW1, SW2: SW_Push, Button_Switch_THT:SW_PUSH_6mm_H5mm
- removed U1: L7805, Package_TO_SOT_SMD:TO-252-3_TabPin2
- removed U2: ESP32-DEVKIT-V1, ESP32-DEVKIT-V1:MODULE_ESP32_DEVKIT_V1
- removed U3, U4: DRV8833, DRV8833:DRV8833
- added BZ7: Buzzer, Buzzer_Beeper:MagneticBuzzer_ProSignal_ABI-009-RC, F.Cu at (139.4, 137.6)
- added C13: 0.33u, Capacitor_SMD:C_1206_3216Metric_Pad1.33x1.80mm_HandSolder, B.Cu at (138.4, 184.0)
- added C14: 0.1u, Capacitor_SMD:C_1206_3216Metric_Pad1.33x1.80mm_HandSolder, B.Cu at (143.5, 184.0)
- added D7: LED_RED, LED_SMD:LED_1206_3216Metric_Pad1.42x1.75mm_HandSolder, F.Cu at (148.2, 191.1)
- added G***16: LOGO, LOGO, F.Cu at (109.8, 195.6)
- added G***17: LOGO, LOGO, F.Cu at (139.4, 195.4)
- added G***18: LOGO, LOGO, F.Cu at (143.2, 125.2)
- added H25: MountingHole, MountingHole:MountingHole_3mm, F.Cu at (105.6, 209.1)
- added H26: MountingHole, MountingHole:MountingHole_3mm, F.Cu at (105.6, 120.6)
- added H27: MountingHole, MountingHole:MountingHole_3mm, F.Cu at (161.0, 209.1)
- added H28: MountingHole, MountingHole:MountingHole_3mm, F.Cu at (161.0, 120.5)
- added J31: M2, TerminalBlock_Phoenix:TerminalBlock_Phoenix_MKDS-1,5-2_1x02_P5.00mm_Horizontal, F.Cu at (124.1, 123.0)
- added J32: SENSORES, Connector_PinHeader_2.54mm:PinHeader_1x11_P2.54mm_Vertical, F.Cu at (156.5, 152.0)
- added R43: 0, Resistor_SMD:R_1206_3216Metric_Pad1.30x1.75mm_HandSolder, B.Cu at (152.2, 184.0)
- added R44: 10k, Resistor_SMD:R_1206_3216Metric_Pad1.30x1.75mm_HandSolder, B.Cu at (114.1, 137.2)
- added R45: 10k, Resistor_SMD:R_1206_3216Metric_Pad1.30x1.75mm_HandSolder, B.Cu at (114.1, 132.2)
- added R46: 220, Resistor_SMD:R_1206_3216Metric_Pad1.30x1.75mm_HandSolder, B.Cu at (148.2, 185.5)
- added R47: 0, Resistor_SMD:R_1206_3216Metric_Pad1.30x1.75mm_HandSolder, B.Cu at (126.7, 181.3)
- added R48: 0, Resistor_SMD:R_1206_3216Metric_Pad1.30x1.75mm_HandSolder, B.Cu at (126.7, 148.2)
- added R49: 0, Resistor_SMD:R_1206_3216Metric_Pad1.30x1.75mm_HandSolder, B.Cu at (137.9, 148.3)
- added SW13: SW_Push, Button_Switch_THT:SW_PUSH_6mm_H5mm, F.Cu at (107.0, 145.5)
- added SW14: SW_Push, Button_Switch_THT:SW_PUSH_6mm_H5mm, F.Cu at (107.0, 130.4)
- added U25: L7805, Package_TO_SOT_SMD:TO-252-3_TabPin2, B.Cu at (141.0, 192.3)
- added U26: ESP32-DEVKIT-V1, ESP32-DEVKIT-V1:MODULE_ESP32_DEVKIT_V1, F.Cu at (129.0, 164.8)
- added U27: DRV8833, DRV8833:DRV8833, F.Cu at (113.0, 191.9)
- added U28: DRV8833, DRV8833:DRV8833, F.Cu at (132.8, 137.6)
- J11: value BAT -> SWITCH; footprint TerminalBlock_Phoenix:TerminalBlock_Phoenix_MKDS-1,5-2_1x02_P5.00mm_Horizontal -> Connector_PinHeader_2.54mm:PinHeader_1x03_P2.54mm_Vertical
- J12: value SWITCH -> M1; footprint Connector_PinHeader_2.54mm:PinHeader_1x03_P2.54mm_Vertical -> TerminalBlock_Phoenix:TerminalBlock_Phoenix_MKDS-1,5-2_1x02_P5.00mm_Horizontal
- J13: value M1 -> M2
- J14: value M2 -> SENSORES; footprint TerminalBlock_Phoenix:TerminalBlock_Phoenix_MKDS-1,5-2_1x02_P5.00mm_Horizontal -> Connector_PinHeader_2.54mm:PinHeader_1x11_P2.54mm_Vertical
- J15: value SENSORES -> SWITCH; footprint Connector_PinHeader_2.54mm:PinHeader_1x11_P2.54mm_Vertical -> Connector_PinHeader_2.54mm:PinHeader_1x03_P2.54mm_Vertical
- J16: value BAT -> M1
- J17: value SWITCH -> M2; footprint Connector_PinHeader_2.54mm:PinHeader_1x03_P2.54mm_Vertical -> TerminalBlock_Phoenix:TerminalBlock_Phoenix_MKDS-1,5-2_1x02_P5.00mm_Horizontal
- J18: value M1 -> SENSORES; footprint TerminalBlock_Phoenix:TerminalBlock_Phoenix_MKDS-1,5-2_1x02_P5.00mm_Horizontal -> Connector_PinHeader_2.54mm:PinHeader_1x11_P2.54mm_Vertical
- J19, J24, J29: value M2 -> SWITCH; footprint TerminalBlock_Phoenix:TerminalBlock_Phoenix_MKDS-1,5-2_1x02_P5.00mm_Horizontal -> Connector_PinHeader_2.54mm:PinHeader_1x03_P2.54mm_Vertical
- J20, J25, J30: value SENSORES -> M1; footprint Connector_PinHeader_2.54mm:PinHeader_1x11_P2.54mm_Vertical -> TerminalBlock_Phoenix:TerminalBlock_Phoenix_MKDS-1,5-2_1x02_P5.00mm_Horizontal
- J21, J26: value BAT -> M2
- J22, J27: value SWITCH -> SENSORES; footprint Connector_PinHeader_2.54mm:PinHeader_1x03_P2.54mm_Vertical -> Connector_PinHeader_2.54mm:PinHeader_1x11_P2.54mm_Vertical
- J23, J28, J4: value M1 -> BAT
- J5: value M2 -> BAT
- J6: value SENSORES -> BAT; footprint Connector_PinHeader_2.54mm:PinHeader_1x11_P2.54mm_Vertical -> TerminalBlock_Phoenix:TerminalBlock_Phoenix_MKDS-1,5-2_1x02_P5.00mm_Horizontal
- moved J22 232.3 mm to (246.5, 47.0), turned to 0 degrees
- moved J21 224.7 mm to (214.1, 18.0), turned to 180 degrees
- moved BZ2 208.4 mm to (229.4, 137.6)
- moved C3 208.4 mm to (228.4, 184.0)
- moved C4 208.4 mm to (233.5, 184.0)
- moved D2 208.4 mm to (238.2, 191.1)
- moved G***1 208.4 mm to (199.8, 195.6)
- moved G***2 208.4 mm to (229.4, 195.4)
- moved G***3 208.4 mm to (233.2, 125.2)
- moved H5 208.4 mm to (195.6, 209.1)
- moved H6 208.4 mm to (195.6, 120.6)
- moved H7 208.4 mm to (251.0, 209.1)
- moved H8 208.4 mm to (251.0, 120.5)
- moved J10 208.4 mm to (246.5, 152.0)
- moved J3 208.4 mm to (246.7, 189.0)
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Connections:
- J11 pad 2: GND -> Net-(J1-Pin_1)
- J12 pad 1: Net-(J1-Pin_1) -> Net-(J4-Pin_1)
- J12 pad 2: Net-(J1-Pin_1) -> Net-(J4-Pin_2)
- J13 pad 1: Net-(J4-Pin_1) -> Net-(J5-Pin_1)
- J13 pad 2: Net-(J4-Pin_2) -> Net-(J5-Pin_2)
- J14 pad 1: Net-(J5-Pin_1) -> +3.3V
- J14 pad 2: Net-(J5-Pin_2) -> /S8
- J15 pad 1: +3.3V -> Net-(J1-Pin_1)
- J15 pad 2: /S8 -> Net-(J1-Pin_1)
- J15 pad 3: /S7 -> VCC
- J16 pad 1: Net-(J1-Pin_1) -> Net-(J4-Pin_1)
- J16 pad 2: GND -> Net-(J4-Pin_2)
- J17 pad 1: Net-(J1-Pin_1) -> Net-(J5-Pin_1)
- J17 pad 2: Net-(J1-Pin_1) -> Net-(J5-Pin_2)
- J18 pad 1: Net-(J4-Pin_1) -> +3.3V
- J18 pad 2: Net-(J4-Pin_2) -> /S8
- J19 pad 1: Net-(J5-Pin_1) -> Net-(J1-Pin_1)
- J19 pad 2: Net-(J5-Pin_2) -> Net-(J1-Pin_1)
- J20 pad 1: +3.3V -> Net-(J4-Pin_1)
- J20 pad 2: /S8 -> Net-(J4-Pin_2)
- J21 pad 1: Net-(J1-Pin_1) -> Net-(J5-Pin_1)
- J21 pad 2: GND -> Net-(J5-Pin_2)
- J22 pad 1: Net-(J1-Pin_1) -> +3.3V
- J22 pad 2: Net-(J1-Pin_1) -> /S8
- J22 pad 3: VCC -> /S7
- J23 pad 1: Net-(J4-Pin_1) -> Net-(J1-Pin_1)
- J23 pad 2: Net-(J4-Pin_2) -> GND
- J24 pad 1: Net-(J5-Pin_1) -> Net-(J1-Pin_1)
- J24 pad 2: Net-(J5-Pin_2) -> Net-(J1-Pin_1)
- J25 pad 1: +3.3V -> Net-(J4-Pin_1)
- J25 pad 2: /S8 -> Net-(J4-Pin_2)
- J26 pad 1: Net-(J1-Pin_1) -> Net-(J5-Pin_1)
- J26 pad 2: GND -> Net-(J5-Pin_2)
- J27 pad 1: Net-(J1-Pin_1) -> +3.3V
- J27 pad 2: Net-(J1-Pin_1) -> /S8
- J27 pad 3: VCC -> /S7
- J28 pad 1: Net-(J4-Pin_1) -> Net-(J1-Pin_1)
- J28 pad 2: Net-(J4-Pin_2) -> GND
- J29 pad 1: Net-(J5-Pin_1) -> Net-(J1-Pin_1)
- J29 pad 2: Net-(J5-Pin_2) -> Net-(J1-Pin_1)
- J30 pad 1: +3.3V -> Net-(J4-Pin_1)
- J30 pad 2: /S8 -> Net-(J4-Pin_2)
- J4 pad 1: Net-(J4-Pin_1) -> Net-(J1-Pin_1)
- J4 pad 2: Net-(J4-Pin_2) -> GND
- J5 pad 1: Net-(J5-Pin_1) -> Net-(J1-Pin_1)
- J5 pad 2: Net-(J5-Pin_2) -> GND
- J6 pad 1: +3.3V -> Net-(J1-Pin_1)
- J6 pad 2: /S8 -> GND
Other:
- board size 238 x 198.6 mm -> 242 x 200 mm
