File: Fabricacion/MATRIZ_COCHE_COMPETENCIA.kicad_pcb (KiCad board)
At the start: 2 copper layers, 242 x 200 mm, 174 parts, among them J10 SENSORES, J11 SWITCH, J12 M1, J13 M2, J14 SENSORES, J15 SWITCH, J16 M1, J17 M2, J18 SENSORES, J19 SWITCH, J20 M1, J21 M2, J22 SENSORES, J23 BAT, J24 SWITCH, J25 M1, J26 M2, J27 SENSORES, J28 BAT, J29 SWITCH, J3 BAT, J30 M1, J31 M2, J32 SENSORES, J4 BAT, J5 BAT, J6 BAT, J7 SWITCH, J8 M1, J9 M2, SW10 SW_Push, SW11 SW_Push, SW12 SW_Push, SW13 SW_Push, SW14 SW_Push, SW3 SW_Push, SW4 SW_Push, SW5 SW_Push, SW6 SW_Push, SW7 SW_Push, SW8 SW_Push, SW9 SW_Push, U10 ESP32-DEVKIT-V1, U11 DRV8833, U12 DRV8833, U13 L7805, U14 ESP32-DEVKIT-V1, U15 DRV8833, U16 DRV8833, U17 L7805, U18 ESP32-DEVKIT-V1, U19 DRV8833, U20 DRV8833, U21 L7805, U22 ESP32-DEVKIT-V1, U23 DRV8833, U24 DRV8833, U25 L7805, U26 ESP32-DEVKIT-V1, U27 DRV8833, U28 DRV8833, U5 L7805, U6 ESP32-DEVKIT-V1, U7 DRV8833, U8 DRV8833, U9 L7805

Commit message: V1.3 - Diodo de proteccion + Mejor ubicacion de Sw's
Parts:
- removed BZ2, BZ3, BZ4: Buzzer, Buzzer_Beeper:MagneticBuzzer_ProSignal_ABI-009-RC
- removed C10, C12, C14, C4, C6, C8: 0.1u, Capacitor_SMD:C_1206_3216Metric_Pad1.33x1.80mm_HandSolder
- removed C11, C13, C3, C5, C7, C9: 0.33u, Capacitor_SMD:C_1206_3216Metric_Pad1.33x1.80mm_HandSolder
- removed D2, D3, D4, D5, D6, D7: LED_RED, LED_SMD:LED_1206_3216Metric_Pad1.42x1.75mm_HandSolder
- removed G***1, G***2, G***3, G***4, G***5, G***6, G***7, G***8, G***9: LOGO, LOGO
- removed H10, H11, H12, H13, H14, H15, H16, H5, H6, H7, H8, H9: MountingHole, MountingHole:MountingHole_3mm
- removed J10, J14, J18: SENSORES, Connector_PinHeader_2.54mm:PinHeader_1x11_P2.54mm_Vertical
- removed J11, J15, J19, J7: SWITCH, Connector_PinHeader_2.54mm:PinHeader_1x03_P2.54mm_Vertical
- removed J12, J16, J20, J8: M1, TerminalBlock_Phoenix:TerminalBlock_Phoenix_MKDS-1,5-2_1x02_P5.00mm_Horizontal
- removed J13, J17, J9: M2, TerminalBlock_Phoenix:TerminalBlock_Phoenix_MKDS-1,5-2_1x02_P5.00mm_Horizontal
- removed J3, J6: BAT, TerminalBlock_Phoenix:TerminalBlock_Phoenix_MKDS-1,5-2_1x02_P5.00mm_Horizontal
- removed R10, R16, R17, R23, R24, R9: 10k, Resistor_SMD:R_1206_3216Metric_Pad1.30x1.75mm_HandSolder
- removed R11, R18, R25: 220, Resistor_SMD:R_1206_3216Metric_Pad1.30x1.75mm_HandSolder
- removed R12, R13, R14, R15, R19, R20, R21, R22, R26, R27, R28, R8: 0, Resistor_SMD:R_1206_3216Metric_Pad1.30x1.75mm_HandSolder
- removed SW3, SW4, SW5, SW6, SW7, SW8: SW_Push, Button_Switch_THT:SW_PUSH_6mm_H5mm
- removed U10, U14, U6: ESP32-DEVKIT-V1, ESP32-DEVKIT-V1:MODULE_ESP32_DEVKIT_V1
- removed U11, U12, U15, U16, U7, U8: DRV8833, DRV8833:DRV8833
- removed U13, U17, U5, U9: L7805, Package_TO_SOT_SMD:TO-252-3_TabPin2
- added (+)4: TestPoint, Connector_PinHeader_2.54mm:PinHeader_1x01_P2.54mm_Vertical, F.Cu at (65.5, 186.1)
- added (+)5: TestPoint, Connector_PinHeader_2.54mm:PinHeader_1x01_P2.54mm_Vertical, F.Cu at (157.5, 186.1)
- added (+)6: TestPoint, Connector_PinHeader_2.54mm:PinHeader_1x01_P2.54mm_Vertical, F.Cu at (249.5, 186.1)
- added (+)7: TestPoint, Connector_PinHeader_2.54mm:PinHeader_1x01_P2.54mm_Vertical, F.Cu at (65.5, 83.1)
- added (+)8: TestPoint, Connector_PinHeader_2.54mm:PinHeader_1x01_P2.54mm_Vertical, F.Cu at (157.5, 83.1)
- added (+)9: TestPoint, Connector_PinHeader_2.54mm:PinHeader_1x01_P2.54mm_Vertical, F.Cu at (249.5, 83.1)
- added (-)4: TestPoint, Connector_PinHeader_2.54mm:PinHeader_1x01_P2.54mm_Vertical, F.Cu at (65.5, 181.1)
- added (-)5: TestPoint, Connector_PinHeader_2.54mm:PinHeader_1x01_P2.54mm_Vertical, F.Cu at (157.5, 181.1)
- added (-)6: TestPoint, Connector_PinHeader_2.54mm:PinHeader_1x01_P2.54mm_Vertical, F.Cu at (249.5, 181.1)
- added (-)7: TestPoint, Connector_PinHeader_2.54mm:PinHeader_1x01_P2.54mm_Vertical, F.Cu at (65.5, 78.1)
- added (-)8: TestPoint, Connector_PinHeader_2.54mm:PinHeader_1x01_P2.54mm_Vertical, F.Cu at (157.5, 78.1)
- added (-)9: TestPoint, Connector_PinHeader_2.54mm:PinHeader_1x01_P2.54mm_Vertical, F.Cu at (249.5, 78.1)
- added BZ10: Buzzer, Buzzer_Beeper:MagneticBuzzer_ProSignal_ABI-009-RC, F.Cu at (253.7, 35.8)
- added BZ8: Buzzer, Buzzer_Beeper:MagneticBuzzer_ProSignal_ABI-009-RC, F.Cu at (69.7, 35.8)
- added BZ9: Buzzer, Buzzer_Beeper:MagneticBuzzer_ProSignal_ABI-009-RC, F.Cu at (161.7, 35.8)
- added C17: 0.33u, Capacitor_SMD:C_1206_3216Metric_Pad1.33x1.80mm_HandSolder, B.Cu at (62.5, 189.5)
- added C18: 0.1u, Capacitor_SMD:C_1206_3216Metric_Pad1.33x1.80mm_HandSolder, B.Cu at (57.8, 195.8)
- added C19: 0.1u, Capacitor_SMD:C_1206_3216Metric_Pad1.33x1.80mm_HandSolder, B.Cu at (33.0, 138.2)
- added C20: 0.1u, Capacitor_SMD:C_1206_3216Metric_Pad1.33x1.80mm_HandSolder, B.Cu at (27.5, 132.7)
- added C21: 0.33u, Capacitor_SMD:C_1206_3216Metric_Pad1.33x1.80mm_HandSolder, B.Cu at (154.5, 189.5)
- added C22: 0.1u, Capacitor_SMD:C_1206_3216Metric_Pad1.33x1.80mm_HandSolder, B.Cu at (149.8, 195.8)
- added C23: 0.1u, Capacitor_SMD:C_1206_3216Metric_Pad1.33x1.80mm_HandSolder, B.Cu at (125.0, 138.2)
- added C24: 0.1u, Capacitor_SMD:C_1206_3216Metric_Pad1.33x1.80mm_HandSolder, B.Cu at (119.5, 132.7)
- added C25: 0.33u, Capacitor_SMD:C_1206_3216Metric_Pad1.33x1.80mm_HandSolder, B.Cu at (246.5, 189.5)
- added C26: 0.1u, Capacitor_SMD:C_1206_3216Metric_Pad1.33x1.80mm_HandSolder, B.Cu at (241.8, 195.8)
- added C27: 0.1u, Capacitor_SMD:C_1206_3216Metric_Pad1.33x1.80mm_HandSolder, B.Cu at (217.0, 138.2)
- added C28: 0.1u, Capacitor_SMD:C_1206_3216Metric_Pad1.33x1.80mm_HandSolder, B.Cu at (211.5, 132.7)
- added C29: 0.33u, Capacitor_SMD:C_1206_3216Metric_Pad1.33x1.80mm_HandSolder, B.Cu at (62.5, 86.5)
- added C30: 0.1u, Capacitor_SMD:C_1206_3216Metric_Pad1.33x1.80mm_HandSolder, B.Cu at (57.8, 92.8)
- added C31: 0.1u, Capacitor_SMD:C_1206_3216Metric_Pad1.33x1.80mm_HandSolder, B.Cu at (33.0, 35.2)
- added C32: 0.1u, Capacitor_SMD:C_1206_3216Metric_Pad1.33x1.80mm_HandSolder, B.Cu at (27.5, 29.7)
- added C33: 0.33u, Capacitor_SMD:C_1206_3216Metric_Pad1.33x1.80mm_HandSolder, B.Cu at (154.5, 86.5)
- added C34: 0.1u, Capacitor_SMD:C_1206_3216Metric_Pad1.33x1.80mm_HandSolder, B.Cu at (149.8, 92.8)
- added C35: 0.1u, Capacitor_SMD:C_1206_3216Metric_Pad1.33x1.80mm_HandSolder, B.Cu at (125.0, 35.2)
- added C36: 0.1u, Capacitor_SMD:C_1206_3216Metric_Pad1.33x1.80mm_HandSolder, B.Cu at (119.5, 29.7)
- added C37: 0.33u, Capacitor_SMD:C_1206_3216Metric_Pad1.33x1.80mm_HandSolder, B.Cu at (246.5, 86.5)
- added C38: 0.1u, Capacitor_SMD:C_1206_3216Metric_Pad1.33x1.80mm_HandSolder, B.Cu at (241.8, 92.8)
- added C39: 0.1u, Capacitor_SMD:C_1206_3216Metric_Pad1.33x1.80mm_HandSolder, B.Cu at (217.0, 35.2)
- added C40: 0.1u, Capacitor_SMD:C_1206_3216Metric_Pad1.33x1.80mm_HandSolder, B.Cu at (211.5, 29.7)
- added D10: 1N4148, Diode_THT:D_DO-35_SOD27_P7.62mm_Horizontal, F.Cu at (60.8, 138.8)
- added D11: LED_RED, LED_THT:LED_D5.0mm, F.Cu at (151.6, 184.0)
- added D12: 1N4148, Diode_THT:D_DO-35_SOD27_P7.62mm_Horizontal, F.Cu at (152.8, 138.8)
- added D13: LED_RED, LED_THT:LED_D5.0mm, F.Cu at (243.6, 184.0)
- added D14: 1N4148, Diode_THT:D_DO-35_SOD27_P7.62mm_Horizontal, F.Cu at (244.8, 138.8)
- added D15: LED_RED, LED_THT:LED_D5.0mm, F.Cu at (59.6, 81.0)
- added D16: 1N4148, Diode_THT:D_DO-35_SOD27_P7.62mm_Horizontal, F.Cu at (60.8, 35.8)
- added D17: LED_RED, LED_THT:LED_D5.0mm, F.Cu at (151.6, 81.0)
- added D18: 1N4148, Diode_THT:D_DO-35_SOD27_P7.62mm_Horizontal, F.Cu at (152.8, 35.8)
- added D19: LED_RED, LED_THT:LED_D5.0mm, F.Cu at (243.6, 81.0)
- added D20: 1N4148, Diode_THT:D_DO-35_SOD27_P7.62mm_Horizontal, F.Cu at (244.8, 35.8)
- added D9: LED_RED, LED_THT:LED_D5.0mm, F.Cu at (59.6, 184.0)
- added G***19: LOGO, LOGO, F.Cu at (59.6, 94.7)
- added G***20: LOGO, LOGO, F.Cu at (27.4, 89.7)
- added G***21: LOGO, LOGO, F.Cu at (32.8, 58.9)
- added G***22: LOGO, LOGO, F.Cu at (151.6, 94.7)
- added G***23: LOGO, LOGO, F.Cu at (119.4, 89.7)
- added G***24: LOGO, LOGO, F.Cu at (124.8, 58.9)
- added G***25: LOGO, LOGO, F.Cu at (243.6, 94.7)
- added G***26: LOGO, LOGO, F.Cu at (211.4, 89.7)
- added G***27: LOGO, LOGO, F.Cu at (216.8, 58.9)
- added H29: MountingHole, MountingHole:MountingHole_3mm, F.Cu at (22.7, 103.1)
- added H30: MountingHole, MountingHole:MountingHole_3mm, F.Cu at (22.7, 14.6)
- added H31: MountingHole, MountingHole:MountingHole_3mm, F.Cu at (78.2, 103.1)
- added H32: MountingHole, MountingHole:MountingHole_3mm, F.Cu at (78.0, 14.6)
- added H33: MountingHole, MountingHole:MountingHole_3mm, F.Cu at (114.7, 103.1)
- added H34: MountingHole, MountingHole:MountingHole_3mm, F.Cu at (114.7, 14.6)
- added H35: MountingHole, MountingHole:MountingHole_3mm, F.Cu at (170.2, 103.1)
- added H36: MountingHole, MountingHole:MountingHole_3mm, F.Cu at (170.0, 14.6)
- added H37: MountingHole, MountingHole:MountingHole_3mm, F.Cu at (206.7, 103.1)
- added H38: MountingHole, MountingHole:MountingHole_3mm, F.Cu at (206.7, 14.6)
- added H39: MountingHole, MountingHole:MountingHole_3mm, F.Cu at (262.2, 103.1)
- added H40: MountingHole, MountingHole:MountingHole_3mm, F.Cu at (262.0, 14.6)
- added J33: M2, TerminalBlock_Phoenix:TerminalBlock_Phoenix_MKDS-1,5-2_1x02_P5.00mm_Horizontal, F.Cu at (228.3, 122.9)
- added J34: SENSORES, Connector_PinHeader_2.54mm:PinHeader_1x11_P2.54mm_Vertical, F.Cu at (258.1, 149.1)
- added J35: SWITCH, Connector_PinHeader_2.54mm:PinHeader_1x03_P2.54mm_Vertical, F.Cu at (74.9, 89.5)
- added J36: M1, TerminalBlock_Phoenix:TerminalBlock_Phoenix_MKDS-1,5-2_1x02_P5.00mm_Horizontal, F.Cu at (44.3, 102.8)
- added J37: M2, TerminalBlock_Phoenix:TerminalBlock_Phoenix_MKDS-1,5-2_1x02_P5.00mm_Horizontal, F.Cu at (44.3, 19.9)
- added J38: SENSORES, Connector_PinHeader_2.54mm:PinHeader_1x11_P2.54mm_Vertical, F.Cu at (74.1, 46.1)
- added J39: BAT, TerminalBlock_Phoenix:TerminalBlock_Phoenix_MKDS-1,5-2_1x02_P5.00mm_Horizontal, F.Cu at (166.1, 83.1)
- added J40: SWITCH, Connector_PinHeader_2.54mm:PinHeader_1x03_P2.54mm_Vertical, F.Cu at (166.9, 89.5)
- added J41: M1, TerminalBlock_Phoenix:TerminalBlock_Phoenix_MKDS-1,5-2_1x02_P5.00mm_Horizontal, F.Cu at (136.3, 102.8)
- added J42: M2, TerminalBlock_Phoenix:TerminalBlock_Phoenix_MKDS-1,5-2_1x02_P5.00mm_Horizontal, F.Cu at (136.3, 19.9)
- added J43: SENSORES, Connector_PinHeader_2.54mm:PinHeader_1x11_P2.54mm_Vertical, F.Cu at (166.1, 46.1)
- added J44: BAT, TerminalBlock_Phoenix:TerminalBlock_Phoenix_MKDS-1,5-2_1x02_P5.00mm_Horizontal, F.Cu at (258.1, 83.1)
- added J45: SWITCH, Connector_PinHeader_2.54mm:PinHeader_1x03_P2.54mm_Vertical, F.Cu at (258.9, 89.5)
- added J46: M1, TerminalBlock_Phoenix:TerminalBlock_Phoenix_MKDS-1,5-2_1x02_P5.00mm_Horizontal, F.Cu at (228.3, 102.8)
- added J47: M2, TerminalBlock_Phoenix:TerminalBlock_Phoenix_MKDS-1,5-2_1x02_P5.00mm_Horizontal, F.Cu at (228.3, 19.9)
- added J48: SENSORES, Connector_PinHeader_2.54mm:PinHeader_1x11_P2.54mm_Vertical, F.Cu at (258.1, 46.1)
- added Q10: 2N3904, Package_TO_SOT_THT:TO-92_Inline_Wide, F.Cu at (235.6, 31.9)
- added Q5: 2N3904, Package_TO_SOT_THT:TO-92_Inline_Wide, F.Cu at (51.6, 134.9)
- added Q6: 2N3904, Package_TO_SOT_THT:TO-92_Inline_Wide, F.Cu at (143.6, 134.9)
- added Q7: 2N3904, Package_TO_SOT_THT:TO-92_Inline_Wide, F.Cu at (235.6, 134.9)
- added Q8: 2N3904, Package_TO_SOT_THT:TO-92_Inline_Wide, F.Cu at (51.6, 31.9)
- added Q9: 2N3904, Package_TO_SOT_THT:TO-92_Inline_Wide, F.Cu at (143.6, 31.9)
- added R50: 0, Resistor_SMD:R_1206_3216Metric_Pad1.30x1.75mm_HandSolder, B.Cu at (75.5, 32.0)
- added R51: 10k, Resistor_SMD:R_1206_3216Metric_Pad1.30x1.75mm_HandSolder, B.Cu at (31.7, 31.3)
- added R52: 10k, Resistor_SMD:R_1206_3216Metric_Pad1.30x1.75mm_HandSolder, B.Cu at (31.7, 26.3)
- added R53: 220, Resistor_SMD:R_1206_3216Metric_Pad1.30x1.75mm_HandSolder, B.Cu at (57.0, 75.8)
- added R54: 0, Resistor_SMD:R_1206_3216Metric_Pad1.30x1.75mm_HandSolder, B.Cu at (44.3, 75.4)
- added R55: 0, Resistor_SMD:R_1206_3216Metric_Pad1.30x1.75mm_HandSolder, B.Cu at (44.2, 42.3)
- added R56: 1k, Resistor_SMD:R_1206_3216Metric_Pad1.30x1.75mm_HandSolder, B.Cu at (54.2, 36.3)
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Connections:
- BZ5 pad 1: Net-(BZ1-+) -> +3.3V
- BZ5 pad 2: GND -> Net-(BZ1--)
- BZ6 pad 1: Net-(BZ1-+) -> +3.3V
- BZ6 pad 2: GND -> Net-(BZ1--)
- BZ7 pad 1: Net-(BZ1-+) -> +3.3V
- BZ7 pad 2: GND -> Net-(BZ1--)
- J21 pad 1: Net-(J5-Pin_1) -> Net-(J1-Pin_1)
- J21 pad 2: Net-(J5-Pin_2) -> Net-(J1-Pin_1)
- J22 pad 1: +3.3V -> Net-(J4-Pin_1)
- J22 pad 2: /S8 -> Net-(J4-Pin_2)
- J23 pad 1: Net-(J1-Pin_1) -> Net-(J5-Pin_1)
- J23 pad 2: GND -> Net-(J5-Pin_2)
- J24 pad 1: Net-(J1-Pin_1) -> +3.3V
- J24 pad 2: Net-(J1-Pin_1) -> /S8
- J24 pad 3: VCC -> /S7
- J25 pad 1: Net-(J4-Pin_1) -> Net-(J1-Pin_1)
- J25 pad 2: Net-(J4-Pin_2) -> GND
- J26 pad 1: Net-(J5-Pin_1) -> Net-(J1-Pin_1)
- J26 pad 2: Net-(J5-Pin_2) -> Net-(J1-Pin_1)
- J27 pad 1: +3.3V -> Net-(J4-Pin_1)
- J27 pad 2: /S8 -> Net-(J4-Pin_2)
- J28 pad 1: Net-(J1-Pin_1) -> Net-(J5-Pin_1)
- J28 pad 2: GND -> Net-(J5-Pin_2)
- J29 pad 1: Net-(J1-Pin_1) -> +3.3V
- J29 pad 2: Net-(J1-Pin_1) -> /S8
- J29 pad 3: VCC -> /S7
- J30 pad 1: Net-(J4-Pin_1) -> Net-(J1-Pin_1)
- J30 pad 2: Net-(J4-Pin_2) -> GND
- J31 pad 1: Net-(J5-Pin_1) -> Net-(J1-Pin_1)
- J31 pad 2: Net-(J5-Pin_2) -> Net-(J1-Pin_1)
- J32 pad 1: +3.3V -> Net-(J4-Pin_1)
- J32 pad 2: /S8 -> Net-(J4-Pin_2)
- R35 pad 2: Net-(BZ1-+) -> Net-(Q1-B)
- R42 pad 2: Net-(BZ1-+) -> Net-(Q1-B)
- R49 pad 2: Net-(BZ1-+) -> Net-(Q1-B)
- U21 pad 1: VCC -> GND
- U21 pad 2: GND -> +5V
- U21 pad 3: +5V -> VCC
- U25 pad 1: VCC -> GND
- U25 pad 2: GND -> +5V
- U25 pad 3: +5V -> VCC
Routing:
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Other:
- board size 242 x 200 mm -> 246 x 198 mm
- board text added: "* MotorBoard FIE * A: Sanchez Samuel * V1.2 - 2025"
- board text added: "ANTENA"
- board text added: "GND IR S1 S2 S3 S4 S5 S6 S7 S8 3.3V"
- board text added: "GND VCC"
- board text added: "USB"
- board text added: "VCC GND"
- board text added: "~S.S - V1.2"
- board text removed: "* MotorBoard FIE * A: Sanchez Samuel * V1.0 - 2025"
- board text removed: "+"
- board text removed: "-"
- board text removed: "3.3V"
- board text removed: "Esto no va a explotar… creo."
- board text removed: "GND"
- board text removed: "IR"
- board text removed: "S1"
- board text removed: "S2"
- board text removed: "S3"
- board text removed: "S4"
- board text removed: "S5"
- board text removed: "S6"
- board text removed: "S7"
- board text removed: "S8"
- board text removed: "V1.0"
- board text removed: "~S.S"

Commit message: V1.3 - Protecciones
Parts:
- removed (+)5, (+)9, (-)5, (-)9: TestPoint, Connector_PinHeader_2.54mm:PinHeader_1x01_P2.54mm_Vertical
- removed BZ10, BZ5, BZ9: Buzzer, Buzzer_Beeper:MagneticBuzzer_ProSignal_ABI-009-RC
- removed C17, C33, C37: 0.33u, Capacitor_SMD:C_1206_3216Metric_Pad1.33x1.80mm_HandSolder
- removed C18, C19, C20, C34, C35, C36, C38, C39, C40: 0.1u, Capacitor_SMD:C_1206_3216Metric_Pad1.33x1.80mm_HandSolder
- removed D13, D15: LED_RED, LED_THT:LED_D5.0mm
- removed D14: 1N4148, Diode_THT:D_DO-35_SOD27_P7.62mm_Horizontal
- removed G***13, G***14, G***15, G***16: LOGO, LOGO
- removed H17, H18, H19, H20, H33, H34, H35, H36, H37, H38, H39, H40: MountingHole, MountingHole:MountingHole_3mm
- removed J21, J45: SWITCH, Connector_PinHeader_2.54mm:PinHeader_1x03_P2.54mm_Vertical
- removed J22, J41, J46: M1, TerminalBlock_Phoenix:TerminalBlock_Phoenix_MKDS-1,5-2_1x02_P5.00mm_Horizontal
- removed J23, J42, J47: M2, TerminalBlock_Phoenix:TerminalBlock_Phoenix_MKDS-1,5-2_1x02_P5.00mm_Horizontal
- removed J24, J43, J48: SENSORES, Connector_PinHeader_2.54mm:PinHeader_1x11_P2.54mm_Vertical
- removed J25, J44: BAT, TerminalBlock_Phoenix:TerminalBlock_Phoenix_MKDS-1,5-2_1x02_P5.00mm_Horizontal
- removed Q10, Q5, Q9: 2N3904, Package_TO_SOT_THT:TO-92_Inline_Wide
- removed R37, R38, R44, R45: 10k, Resistor_SMD:R_1206_3216Metric_Pad1.30x1.75mm_HandSolder
- removed R39: 220, Resistor_SMD:R_1206_3216Metric_Pad1.30x1.75mm_HandSolder
- removed R40, R41, R43: 0, Resistor_SMD:R_1206_3216Metric_Pad1.30x1.75mm_HandSolder
- removed R42: 1k, Resistor_SMD:R_1206_3216Metric_Pad1.30x1.75mm_HandSolder
- removed SW10, SW17, SW18, SW19, SW20, SW9: SW_Push, Button_Switch_THT:SW_PUSH_6mm_H5mm
- removed U18, U34, U38: ESP32-DEVKIT-V1, ESP32-DEVKIT-V1:MODULE_ESP32_DEVKIT_V1
- removed U19, U20, U35, U36, U39, U40: DRV8833, DRV8833:DRV8833
- removed U21, U37, U41: AMS1117, Package_TO_SOT_SMD:SOT-223-3_TabPin2
- added (+)2: TestPoint, Connector_PinHeader_2.54mm:PinHeader_1x01_P2.54mm_Vertical, F.Cu at (245.6, 85.4)
- added (+)3: TestPoint, Connector_PinHeader_2.54mm:PinHeader_1x01_P2.54mm_Vertical, F.Cu at (61.6, 85.4)
- added (-)2: TestPoint, Connector_PinHeader_2.54mm:PinHeader_1x01_P2.54mm_Vertical, F.Cu at (245.6, 80.4)
- added (-)3: TestPoint, Connector_PinHeader_2.54mm:PinHeader_1x01_P2.54mm_Vertical, F.Cu at (61.6, 80.4)
- added BZ2: Buzzer, Buzzer_Beeper:MagneticBuzzer_ProSignal_ABI-009-RC, F.Cu at (249.8, 38.1)
- added BZ3: Buzzer, Buzzer_Beeper:MagneticBuzzer_ProSignal_ABI-009-RC, F.Cu at (65.8, 38.1)
- added BZ4: Buzzer, Buzzer_Beeper:MagneticBuzzer_ProSignal_ABI-009-RC, F.Cu at (157.8, 38.1)
- added C10: 1u, Capacitor_SMD:C_1206_3216Metric_Pad1.33x1.80mm_HandSolder, B.Cu at (55.2, 94.7)
- added C11: 100n, Capacitor_SMD:C_1206_3216Metric_Pad1.33x1.80mm_HandSolder, B.Cu at (30.3, 36.4)
- added C12: 100n, Capacitor_SMD:C_1206_3216Metric_Pad1.33x1.80mm_HandSolder, B.Cu at (30.3, 32.4)
- added C13: 100n, Capacitor_SMD:C_1206_3216Metric_Pad1.33x1.80mm_HandSolder, B.Cu at (152.0, 88.4)
- added C14: 1u, Capacitor_SMD:C_1206_3216Metric_Pad1.33x1.80mm_HandSolder, B.Cu at (147.2, 94.7)
- added C15: 100n, Capacitor_SMD:C_1206_3216Metric_Pad1.33x1.80mm_HandSolder, B.Cu at (122.3, 36.4)
- added C16: 100n, Capacitor_SMD:C_1206_3216Metric_Pad1.33x1.80mm_HandSolder, B.Cu at (122.3, 32.4)
- added C5: 100n, Capacitor_SMD:C_1206_3216Metric_Pad1.33x1.80mm_HandSolder, B.Cu at (244.0, 88.4)
- added C6: 1u, Capacitor_SMD:C_1206_3216Metric_Pad1.33x1.80mm_HandSolder, B.Cu at (239.2, 94.7)
- added C7: 100n, Capacitor_SMD:C_1206_3216Metric_Pad1.33x1.80mm_HandSolder, B.Cu at (214.3, 36.4)
- added C8: 100n, Capacitor_SMD:C_1206_3216Metric_Pad1.33x1.80mm_HandSolder, B.Cu at (214.3, 32.4)
- added C9: 100n, Capacitor_SMD:C_1206_3216Metric_Pad1.33x1.80mm_HandSolder, B.Cu at (60.0, 88.4)
- added D21: 1N5822, Diode_THT:D_DO-201AD_P12.70mm_Horizontal, F.Cu at (55.5, 200.3)
- added D22: LED_RED, LED_THT:LED_D5.0mm, F.Cu at (144.5, 186.5)
- added D23: 1N4148, Diode_THT:D_DO-35_SOD27_P7.62mm_Horizontal, F.Cu at (148.9, 138.1)
- added D24: 1N5822, Diode_THT:D_DO-201AD_P12.70mm_Horizontal, F.Cu at (147.5, 200.3)
- added D4: LED_RED, LED_THT:LED_D5.0mm, F.Cu at (236.5, 86.5)
- added D5: 1N4148, Diode_THT:D_DO-35_SOD27_P7.62mm_Horizontal, F.Cu at (240.9, 38.1)
- added D6: 1N5822, Diode_THT:D_DO-201AD_P12.70mm_Horizontal, F.Cu at (239.5, 100.3)
- added D7: LED_RED, LED_THT:LED_D5.0mm, F.Cu at (52.5, 86.5)
- added D8: 1N4148, Diode_THT:D_DO-35_SOD27_P7.62mm_Horizontal, F.Cu at (56.9, 38.1)
- added G***1: LOGO, LOGO, B.Cu at (206.6, 98.0)
- added G***2: LOGO, LOGO, F.Cu at (207.5, 91.9)
- added G***28: LOGO, LOGO, F.Cu at (121.0, 161.2)
- added G***3: LOGO, LOGO, F.Cu at (236.2, 87.8)
- added G***4: LOGO, LOGO, F.Cu at (213.0, 61.2)
- added G***5: LOGO, LOGO, B.Cu at (22.6, 98.0)
- added G***6: LOGO, LOGO, F.Cu at (23.5, 91.9)
- added G***7: LOGO, LOGO, F.Cu at (52.2, 87.8)
- added G***8: LOGO, LOGO, F.Cu at (29.0, 61.2)
- added G***9: LOGO, LOGO, B.Cu at (114.6, 98.0)
- added H10: MountingHole, MountingHole:MountingHole_3mm, F.Cu at (18.8, 16.9)
- added H11: MountingHole, MountingHole:MountingHole_3mm, F.Cu at (74.3, 105.4)
- added H12: MountingHole, MountingHole:MountingHole_3mm, F.Cu at (74.2, 16.9)
- added H13: MountingHole, MountingHole:MountingHole_3mm, F.Cu at (110.8, 105.4)
- added H14: MountingHole, MountingHole:MountingHole_3mm, F.Cu at (110.8, 16.9)
- added H15: MountingHole, MountingHole:MountingHole_3mm, F.Cu at (166.3, 105.4)
- added H16: MountingHole, MountingHole:MountingHole_3mm, F.Cu at (166.2, 16.9)
- added H5: MountingHole, MountingHole:MountingHole_3mm, F.Cu at (202.8, 105.4)
- added H6: MountingHole, MountingHole:MountingHole_3mm, F.Cu at (202.8, 16.9)
- added H7: MountingHole, MountingHole:MountingHole_3mm, F.Cu at (258.3, 105.4)
- added H8: MountingHole, MountingHole:MountingHole_3mm, F.Cu at (258.2, 16.9)
- added H9: MountingHole, MountingHole:MountingHole_3mm, F.Cu at (18.8, 105.4)
- added J10: SENSORES, Connector_PinHeader_2.54mm:PinHeader_1x11_P2.54mm_Vertical, F.Cu at (254.2, 48.4)
- added J11: SWITCH, Connector_PinHeader_2.54mm:PinHeader_1x03_P2.54mm_Vertical, F.Cu at (71.0, 91.8)
- added J12: M1, TerminalBlock_Phoenix:TerminalBlock_Phoenix_MKDS-1,5-2_1x02_P5.00mm_Horizontal, F.Cu at (40.4, 105.1)
- added J13: M2, TerminalBlock_Phoenix:TerminalBlock_Phoenix_MKDS-1,5-2_1x02_P5.00mm_Horizontal, F.Cu at (40.4, 22.2)
- added J14: SENSORES, Connector_PinHeader_2.54mm:PinHeader_1x11_P2.54mm_Vertical, F.Cu at (70.2, 48.4)
- added J15: SWITCH, Connector_PinHeader_2.54mm:PinHeader_1x03_P2.54mm_Vertical, F.Cu at (163.0, 91.8)
- added J16: M1, TerminalBlock_Phoenix:TerminalBlock_Phoenix_MKDS-1,5-2_1x02_P5.00mm_Horizontal, F.Cu at (132.4, 105.1)
- added J17: M2, TerminalBlock_Phoenix:TerminalBlock_Phoenix_MKDS-1,5-2_1x02_P5.00mm_Horizontal, F.Cu at (132.4, 22.2)
- added J18: SENSORES, Connector_PinHeader_2.54mm:PinHeader_1x11_P2.54mm_Vertical, F.Cu at (162.2, 48.4)
- added J3: BAT, TerminalBlock_Phoenix:TerminalBlock_Phoenix_MKDS-1,5-2_1x02_P5.00mm_Horizontal, F.Cu at (254.2, 85.4)
- added J7: SWITCH, Connector_PinHeader_2.54mm:PinHeader_1x03_P2.54mm_Vertical, F.Cu at (255.0, 91.8)
- added J8: M1, TerminalBlock_Phoenix:TerminalBlock_Phoenix_MKDS-1,5-2_1x02_P5.00mm_Horizontal, F.Cu at (224.4, 105.1)
- added J9: M2, TerminalBlock_Phoenix:TerminalBlock_Phoenix_MKDS-1,5-2_1x02_P5.00mm_Horizontal, F.Cu at (224.4, 22.2)
- added Q2: 2N3904, Package_TO_SOT_THT:TO-92_Inline_Wide, F.Cu at (231.8, 34.2)
- added Q3: 2N3904, Package_TO_SOT_THT:TO-92_Inline_Wide, F.Cu at (47.8, 34.2)
- added Q4: 2N3904, Package_TO_SOT_THT:TO-92_Inline_Wide, F.Cu at (139.8, 34.2)
- added R10: 0, Resistor_SMD:R_1206_3216Metric_Pad1.30x1.75mm_HandSolder, B.Cu at (255.6, 34.3)
- added R11: 10k, Resistor_SMD:R_1206_3216Metric_Pad1.30x1.75mm_HandSolder, B.Cu at (214.3, 38.7)
- added R12: 10k, Resistor_SMD:R_1206_3216Metric_Pad1.30x1.75mm_HandSolder, B.Cu at (214.3, 30.1)
- added R13: 220, Resistor_SMD:R_1206_3216Metric_Pad1.30x1.75mm_HandSolder, B.Cu at (238.0, 83.9)
- added R14: 0, Resistor_SMD:R_1206_3216Metric_Pad1.30x1.75mm_HandSolder, B.Cu at (224.4, 77.7)
- added R15: 0, Resistor_SMD:R_1206_3216Metric_Pad1.30x1.75mm_HandSolder, B.Cu at (224.4, 44.6)
- added R16: 1k, Resistor_SMD:R_1206_3216Metric_Pad1.30x1.75mm_HandSolder, B.Cu at (234.3, 38.6)
- added R17: 100, Resistor_SMD:R_1206_3216Metric_Pad1.30x1.75mm_HandSolder, B.Cu at (210.8, 22.9)
- added R18: 100, Resistor_SMD:R_1206_3216Metric_Pad1.30x1.75mm_HandSolder, B.Cu at (210.7, 45.2)
- added R19: 0, Resistor_SMD:R_1206_3216Metric_Pad1.30x1.75mm_HandSolder, B.Cu at (71.6, 34.3)
- added R20: 10k, Resistor_SMD:R_1206_3216Metric_Pad1.30x1.75mm_HandSolder, B.Cu at (30.3, 38.7)
- added R21: 10k, Resistor_SMD:R_1206_3216Metric_Pad1.30x1.75mm_HandSolder, B.Cu at (30.3, 30.1)
- added R22: 220, Resistor_SMD:R_1206_3216Metric_Pad1.30x1.75mm_HandSolder, B.Cu at (54.0, 83.9)
- added R23: 0, Resistor_SMD:R_1206_3216Metric_Pad1.30x1.75mm_HandSolder, B.Cu at (40.4, 77.7)
- added R24: 0, Resistor_SMD:R_1206_3216Metric_Pad1.30x1.75mm_HandSolder, B.Cu at (40.4, 44.6)
- added R25: 1k, Resistor_SMD:R_1206_3216Metric_Pad1.30x1.75mm_HandSolder, B.Cu at (50.3, 38.6)
- added R26: 100, Resistor_SMD:R_1206_3216Metric_Pad1.30x1.75mm_HandSolder, B.Cu at (26.8, 22.9)
- added R27: 100, Resistor_SMD:R_1206_3216Metric_Pad1.30x1.75mm_HandSolder, B.Cu at (26.7, 45.2)
- added R28: 0, Resistor_SMD:R_1206_3216Metric_Pad1.30x1.75mm_HandSolder, B.Cu at (163.6, 34.3)
- added R71: 100, Resistor_SMD:R_1206_3216Metric_Pad1.30x1.75mm_HandSolder, B.Cu at (118.8, 122.9)
- added R72: 100, Resistor_SMD:R_1206_3216Metric_Pad1.30x1.75mm_HandSolder, B.Cu at (118.7, 145.2)
- added SW3: SW_Push, Button_Switch_THT:SW_PUSH_6mm_H5mm, F.Cu at (209.7, 41.9)
- added SW4: SW_Push, Button_Switch_THT:SW_PUSH_6mm_H5mm, F.Cu at (203.2, 26.9)
- added SW5: SW_Push, Button_Switch_THT:SW_PUSH_6mm_H5mm, F.Cu at (25.7, 41.9)
- added SW6: SW_Push, Button_Switch_THT:SW_PUSH_6mm_H5mm, F.Cu at (19.2, 26.9)
- added SW7: SW_Push, Button_Switch_THT:SW_PUSH_6mm_H5mm, F.Cu at (117.7, 41.9)
- added SW8: SW_Push, Button_Switch_THT:SW_PUSH_6mm_H5mm, F.Cu at (111.2, 26.9)
- added U10: ESP32-DEVKIT-V1, ESP32-DEVKIT-V1:MODULE_ESP32_DEVKIT_V1, F.Cu at (42.7, 61.2)
- added U11: DRV8833, DRV8833:DRV8833, F.Cu at (26.7, 88.3)
- added U12: DRV8833, DRV8833:DRV8833, F.Cu at (46.5, 34.0)
- added U13: AMS1117, Package_TO_SOT_SMD:SOT-223-3_TabPin2, B.Cu at (60.0, 94.6)
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Connections:
- C23 pad 1: /SW1 -> Net-(C3-Pad1)
- C24 pad 1: /SW2 -> Net-(C4-Pad1)
- C27 pad 1: /SW1 -> Net-(C3-Pad1)
- C28 pad 1: /SW2 -> Net-(C4-Pad1)
- C31 pad 1: /SW1 -> Net-(C3-Pad1)
- C32 pad 1: /SW2 -> Net-(C4-Pad1)
- D10 pad 1: +3.3V -> Net-(D1-K)
- D10 pad 2: Net-(BZ1--) -> /LED_LARGADA
- D11 pad 1: GND -> +3.3V
- D11 pad 2: Net-(D1-A) -> Net-(BZ1--)
- D12 pad 1: +3.3V -> VCC
- D12 pad 2: Net-(BZ1--) -> Net-(D3-A)
- D16 pad 1: +3.3V -> Net-(D1-K)
- D16 pad 2: Net-(BZ1--) -> /LED_LARGADA
- D17 pad 1: GND -> +3.3V
- D17 pad 2: Net-(D1-A) -> Net-(BZ1--)
- D18 pad 1: +3.3V -> VCC
- D18 pad 2: Net-(BZ1--) -> Net-(D3-A)
- D19 pad 1: GND -> Net-(D1-K)
- D19 pad 2: Net-(D1-A) -> /LED_LARGADA
- D9 pad 1: GND -> VCC
- D9 pad 2: Net-(D1-A) -> Net-(D3-A)
- J26 pad 2: Net-(J1-Pin_1) -> GND
- J27 pad 1: Net-(J4-Pin_1) -> Net-(J1-Pin_1)
- J27 pad 2: Net-(J4-Pin_2) -> Net-(J1-Pin_1)
- J28 pad 1: Net-(J5-Pin_1) -> Net-(J4-Pin_1)
- J28 pad 2: Net-(J5-Pin_2) -> Net-(J4-Pin_2)
- J29 pad 1: +3.3V -> Net-(J5-Pin_1)
- J29 pad 2: /S8 -> Net-(J5-Pin_2)
- J30 pad 1: Net-(J1-Pin_1) -> +3.3V
- J30 pad 2: GND -> /S8
- J31 pad 2: Net-(J1-Pin_1) -> GND
- J32 pad 1: Net-(J4-Pin_1) -> Net-(J1-Pin_1)
- J32 pad 2: Net-(J4-Pin_2) -> Net-(J1-Pin_1)
- J33 pad 1: Net-(J5-Pin_1) -> Net-(J4-Pin_1)
- J33 pad 2: Net-(J5-Pin_2) -> Net-(J4-Pin_2)
- J34 pad 1: +3.3V -> Net-(J5-Pin_1)
- J34 pad 2: /S8 -> Net-(J5-Pin_2)
- J35 pad 1: Net-(J1-Pin_1) -> +3.3V
- J35 pad 2: Net-(J1-Pin_1) -> /S8
- J35 pad 3: VCC -> /S7
- J36 pad 1: Net-(J4-Pin_1) -> Net-(J1-Pin_1)
- J36 pad 2: Net-(J4-Pin_2) -> GND
- J37 pad 1: Net-(J5-Pin_1) -> Net-(J1-Pin_1)
- J37 pad 2: Net-(J5-Pin_2) -> Net-(J1-Pin_1)
- J38 pad 1: +3.3V -> Net-(J4-Pin_1)
- J38 pad 2: /S8 -> Net-(J4-Pin_2)
- J39 pad 1: Net-(J1-Pin_1) -> Net-(J5-Pin_1)
- J39 pad 2: GND -> Net-(J5-Pin_2)
- J40 pad 1: Net-(J1-Pin_1) -> +3.3V
- J40 pad 2: Net-(J1-Pin_1) -> /S8
- J40 pad 3: VCC -> /S7
- R29 pad 1: GND -> Net-(C3-Pad1)
- R30 pad 1: /SW1 -> Net-(C4-Pad1)
- R31 pad 1: /SW2 -> Net-(D1-K)
- R32 pad 1: /LED_LARGADA -> /IN_M1_A
- R32 pad 2: Net-(D1-A) -> Net-(U3-IN2)
- R33 pad 1: /IN_M1_A -> /IN_M2_B
- R33 pad 2: Net-(U3-IN2) -> Net-(U4-IN3)
- R34 pad 1: /IN_M2_B -> /BUZZER
- R34 pad 2: Net-(U4-IN3) -> Net-(Q1-B)
- R35 pad 1: /BUZZER -> Net-(C4-Pad1)
- R35 pad 2: Net-(Q1-B) -> /SW2
- R36 pad 1: GND -> Net-(C3-Pad1)
- R36 pad 2: GND -> /SW1
- R46 pad 1: /LED_LARGADA -> GND
- R46 pad 2: Net-(D1-A) -> GND
- R47 pad 1: /IN_M1_A -> Net-(C3-Pad1)
- R47 pad 2: Net-(U3-IN2) -> GND
- R48 pad 1: /IN_M2_B -> Net-(C4-Pad1)
- R48 pad 2: Net-(U4-IN3) -> GND
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Routing:
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Other:
- board size 246 x 198 mm -> 246 x 195 mm
- board text added: "* MotorBoard FIE * A: Sanchez Samuel * V1.3 - 2025"
- board text added: "2025 - V1.3"
- board text added: "~S.S"
- board text removed: "* MotorBoard FIE * A: Sanchez Samuel * V1.2 - 2025"
- board text removed: "~S.S - V1.2"

Commit message: V1.4 - Mejores pistas & Modulo de Interrupciones
Parts:
- removed (+)7, (+)8, (-)7, (-)8: TestPoint, Connector_PinHeader_2.54mm:PinHeader_1x01_P2.54mm_Vertical
- removed BZ7, BZ8: Buzzer, Buzzer_Beeper:MagneticBuzzer_ProSignal_ABI-009-RC
- removed C25, C27, C28, C29, C31, C32: 100n, Capacitor_SMD:C_1206_3216Metric_Pad1.33x1.80mm_HandSolder
- removed C26, C30: 1u, Capacitor_SMD:C_1206_3216Metric_Pad1.33x1.80mm_HandSolder
- removed D19, D22: LED_RED, LED_THT:LED_D5.0mm
- removed D20, D23: 1N4148, Diode_THT:D_DO-35_SOD27_P7.62mm_Horizontal
- removed D21, D24: 1N5822, Diode_THT:D_DO-201AD_P12.70mm_Horizontal
- removed G***21, G***22, G***23, G***24, G***25, G***26, G***27, G***28: LOGO, LOGO
- removed H25, H26, H27, H28, H29, H30, H31, H32: MountingHole, MountingHole:MountingHole_3mm
- removed J31, J36: BAT, TerminalBlock_Phoenix:TerminalBlock_Phoenix_MKDS-1,5-2_1x02_P5.00mm_Horizontal
- removed J32, J37: SWITCH, Connector_PinHeader_2.54mm:PinHeader_1x03_P2.54mm_Vertical
- removed J33, J38: M1, TerminalBlock_Phoenix:TerminalBlock_Phoenix_MKDS-1,5-2_1x02_P5.00mm_Horizontal
- removed J34, J39: M2, TerminalBlock_Phoenix:TerminalBlock_Phoenix_MKDS-1,5-2_1x02_P5.00mm_Horizontal
- removed J35, J40: SENSORES, Connector_PinHeader_2.54mm:PinHeader_1x11_P2.54mm_Vertical
- removed Q7, Q8: 2N3904, Package_TO_SOT_THT:TO-92_Inline_Wide
- removed R50, R51, R55, R59, R60, R64, R68, R69: 0, Resistor_SMD:R_1206_3216Metric_Pad1.30x1.75mm_HandSolder
- removed R52, R61, R70: 1k, Resistor_SMD:R_1206_3216Metric_Pad1.30x1.75mm_HandSolder
- removed R53, R54, R62, R63, R71, R72: 100, Resistor_SMD:R_1206_3216Metric_Pad1.30x1.75mm_HandSolder
- removed R56, R57, R65, R66: 10k, Resistor_SMD:R_1206_3216Metric_Pad1.30x1.75mm_HandSolder
- removed R58, R67: 220, Resistor_SMD:R_1206_3216Metric_Pad1.30x1.75mm_HandSolder
- removed SW13, SW14, SW15, SW16: SW_Push, Button_Switch_THT:SW_PUSH_6mm_H5mm
- removed U26, U30: ESP32-DEVKIT-V1, ESP32-DEVKIT-V1:MODULE_ESP32_DEVKIT_V1
- removed U27, U28, U31, U32: DRV8833, DRV8833:DRV8833
- removed U29, U33: AMS1117, Package_TO_SOT_SMD:SOT-223-3_TabPin2
- added (+)1: TestPoint, Connector_PinHeader_2.54mm:PinHeader_1x01_P2.54mm_Vertical, F.Cu at (246.3, 184.0)
- added (+)5: TestPoint, Connector_PinHeader_2.54mm:PinHeader_1x01_P2.54mm_Vertical, F.Cu at (56.3, 184.0)
- added (-)1: TestPoint, Connector_PinHeader_2.54mm:PinHeader_1x01_P2.54mm_Vertical, F.Cu at (246.3, 179.0)
- added (-)5: TestPoint, Connector_PinHeader_2.54mm:PinHeader_1x01_P2.54mm_Vertical, F.Cu at (56.3, 179.0)
- added BZ1: Buzzer, Buzzer_Beeper:MagneticBuzzer_ProSignal_ABI-009-RC, F.Cu at (250.5, 136.7)
- added BZ5: Buzzer, Buzzer_Beeper:MagneticBuzzer_ProSignal_ABI-009-RC, F.Cu at (60.5, 136.7)
- added C1: 100n, Capacitor_SMD:C_1206_3216Metric_Pad1.33x1.80mm_HandSolder, B.Cu at (244.7, 187.0)
- added C17: 100n, Capacitor_SMD:C_1206_3216Metric_Pad1.33x1.80mm_HandSolder, B.Cu at (54.7, 187.0)
- added C18: 1u, Capacitor_SMD:C_1206_3216Metric_Pad1.33x1.80mm_HandSolder, B.Cu at (49.9, 193.3)
- added C19: 100n, Capacitor_SMD:C_1206_3216Metric_Pad1.33x1.80mm_HandSolder, B.Cu at (25.0, 135.0)
- added C2: 1u, Capacitor_SMD:C_1206_3216Metric_Pad1.33x1.80mm_HandSolder, B.Cu at (239.9, 193.3)
- added C20: 100n, Capacitor_SMD:C_1206_3216Metric_Pad1.33x1.80mm_HandSolder, B.Cu at (25.0, 131.2)
- added C3: 100n, Capacitor_SMD:C_1206_3216Metric_Pad1.33x1.80mm_HandSolder, B.Cu at (215.0, 135.0)
- added C4: 100n, Capacitor_SMD:C_1206_3216Metric_Pad1.33x1.80mm_HandSolder, B.Cu at (215.0, 131.2)
- added D1: LED_RED, LED_THT:LED_D5.0mm, F.Cu at (237.2, 185.1)
- added D13: LED_RED, LED_THT:LED_D5.0mm, F.Cu at (47.2, 185.1)
- added D14: 1N4148, Diode_THT:D_DO-35_SOD27_P7.62mm_Horizontal, F.Cu at (50.4, 136.7)
- added D15: 1N5822, Diode_THT:D_DO-201AD_P12.70mm_Horizontal, F.Cu at (50.2, 198.9)
- added D2: 1N4148, Diode_THT:D_DO-35_SOD27_P7.62mm_Horizontal, F.Cu at (240.4, 136.7)
- added D3: 1N5822, Diode_THT:D_DO-201AD_P12.70mm_Horizontal, F.Cu at (240.2, 198.9)
- added G***: LOGO, LOGO, F.Cu at (236.9, 186.3)
- added G***: LOGO, LOGO, F.Cu at (213.7, 159.8)
- added G***: LOGO, LOGO, F.Cu at (208.2, 190.5)
- added G***: LOGO, LOGO, B.Cu at (207.3, 196.6)
- added G***13: LOGO, LOGO, B.Cu at (17.3, 196.6)
- added G***14: LOGO, LOGO, F.Cu at (18.2, 190.5)
- added G***15: LOGO, LOGO, F.Cu at (46.9, 186.3)
- added G***16: LOGO, LOGO, F.Cu at (23.7, 159.8)
- added H1: MountingHole, MountingHole:MountingHole_3mm, F.Cu at (204.8, 204.1)
- added H17: MountingHole, MountingHole:MountingHole_3mm, F.Cu at (14.8, 204.1)
- added H18: MountingHole, MountingHole:MountingHole_3mm, F.Cu at (14.8, 115.5)
- added H19: MountingHole, MountingHole:MountingHole_3mm, F.Cu at (70.4, 204.1)
- added H2: MountingHole, MountingHole:MountingHole_3mm, F.Cu at (204.8, 115.5)
- added H20: MountingHole, MountingHole:MountingHole_3mm, F.Cu at (70.4, 115.5)
- added H3: MountingHole, MountingHole:MountingHole_3mm, F.Cu at (260.4, 204.1)
- added H4: MountingHole, MountingHole:MountingHole_3mm, F.Cu at (260.4, 115.5)
- added J1: BAT, TerminalBlock_Phoenix:TerminalBlock_Phoenix_MKDS-1,5-2_1x02_P5.00mm_Horizontal, F.Cu at (255.0, 184.0)
- added J19: M2, TerminalBlock_Phoenix:TerminalBlock_Phoenix_MKDS-1,5-2_1x02_P5.00mm_Horizontal, F.Cu at (225.1, 18.8)
- added J2: SWITCH, Connector_PinHeader_2.54mm:PinHeader_1x03_P2.54mm_Vertical, F.Cu at (255.7, 190.4)
- added J20: SENSORES, Connector_PinHeader_2.54mm:PinHeader_1x11_P2.54mm_Vertical, F.Cu at (255.0, 45.0)
- added J21: BAT, TerminalBlock_Phoenix:TerminalBlock_Phoenix_MKDS-1,5-2_1x02_P5.00mm_Horizontal, F.Cu at (65.0, 184.0)
- added J22: SWITCH, Connector_PinHeader_2.54mm:PinHeader_1x03_P2.54mm_Vertical, F.Cu at (65.7, 190.4)
- added J23: M1, TerminalBlock_Phoenix:TerminalBlock_Phoenix_MKDS-1,5-2_1x02_P5.00mm_Horizontal, F.Cu at (35.1, 203.6)
- added J24: M2, TerminalBlock_Phoenix:TerminalBlock_Phoenix_MKDS-1,5-2_1x02_P5.00mm_Horizontal, F.Cu at (35.1, 120.8)
- added J25: SENSORES, Connector_PinHeader_2.54mm:PinHeader_1x11_P2.54mm_Vertical, F.Cu at (65.0, 147.0)
- added J6: SENSORES, Connector_PinHeader_2.54mm:PinHeader_1x11_P2.54mm_Vertical, F.Cu at (255.0, 147.0)
- added Q1: 2N3904, Package_TO_SOT_THT:TO-92_Inline_Wide, F.Cu at (235.3, 135.4)
- added Q5: 2N3904, Package_TO_SOT_THT:TO-92_Inline_Wide, F.Cu at (45.3, 135.4)
- added R2: 10k, Resistor_SMD:R_1206_3216Metric_Pad1.30x1.75mm_HandSolder, B.Cu at (215.0, 137.3)
- added R3: 10k, Resistor_SMD:R_1206_3216Metric_Pad1.30x1.75mm_HandSolder, B.Cu at (215.0, 128.9)
- added R37: 0, Resistor_SMD:R_1206_3216Metric_Pad1.30x1.75mm_HandSolder, B.Cu at (35.2, 176.3)
- added R38: 0, Resistor_SMD:R_1206_3216Metric_Pad1.30x1.75mm_HandSolder, B.Cu at (35.1, 143.1)
- added R39: 1k, Resistor_SMD:R_1206_3216Metric_Pad1.30x1.75mm_HandSolder, B.Cu at (44.3, 143.1)
- added R4: 220, Resistor_SMD:R_1206_3216Metric_Pad1.30x1.75mm_HandSolder, B.Cu at (238.7, 182.5)
- added R40: 100, Resistor_SMD:R_1206_3216Metric_Pad1.30x1.75mm_HandSolder, B.Cu at (21.5, 122.6)
- added R41: 100, Resistor_SMD:R_1206_3216Metric_Pad1.30x1.75mm_HandSolder, B.Cu at (21.4, 143.8)
- added R42: 10k, Resistor_SMD:R_1206_3216Metric_Pad1.30x1.75mm_HandSolder, B.Cu at (120.0, 137.3)
- added R43: 10k, Resistor_SMD:R_1206_3216Metric_Pad1.30x1.75mm_HandSolder, B.Cu at (120.0, 128.9)
- added R44: 220, Resistor_SMD:R_1206_3216Metric_Pad1.30x1.75mm_HandSolder, B.Cu at (143.7, 182.5)
- added R45: 0, Resistor_SMD:R_1206_3216Metric_Pad1.30x1.75mm_HandSolder, B.Cu at (130.2, 176.3)
- added R5: 0, Resistor_SMD:R_1206_3216Metric_Pad1.30x1.75mm_HandSolder, B.Cu at (225.2, 176.3)
- added R6: 0, Resistor_SMD:R_1206_3216Metric_Pad1.30x1.75mm_HandSolder, B.Cu at (225.1, 143.1)
- added R7: 1k, Resistor_SMD:R_1206_3216Metric_Pad1.30x1.75mm_HandSolder, B.Cu at (234.3, 143.1)
- added R8: 100, Resistor_SMD:R_1206_3216Metric_Pad1.30x1.75mm_HandSolder, B.Cu at (211.5, 122.6)
- added R9: 100, Resistor_SMD:R_1206_3216Metric_Pad1.30x1.75mm_HandSolder, B.Cu at (211.4, 143.8)
- added SW1: SW_Push, Button_Switch_THT:SW_PUSH_6mm_H5mm, F.Cu at (203.9, 136.0)
- added SW10: SW_Push, Button_Switch_THT:SW_PUSH_6mm_H5mm, F.Cu at (20.4, 129.9)
- added SW2: SW_Push, Button_Switch_THT:SW_PUSH_6mm_H5mm, F.Cu at (210.4, 129.9)
- added SW9: SW_Push, Button_Switch_THT:SW_PUSH_6mm_H5mm, F.Cu at (13.9, 136.0)
- added U18: ESP32-DEVKIT-V1, ESP32-DEVKIT-V1:MODULE_ESP32_DEVKIT_V1, F.Cu at (37.4, 159.8)
- added U19: DRV8833, DRV8833:DRV8833, F.Cu at (21.4, 186.8)
- added U2: ESP32-DEVKIT-V1, ESP32-DEVKIT-V1:MODULE_ESP32_DEVKIT_V1, F.Cu at (227.4, 159.8)
- added U20: DRV8833, DRV8833:DRV8833, F.Cu at (41.2, 132.6)
- added U21: AMS1117, Package_TO_SOT_SMD:SOT-223-3_TabPin2, B.Cu at (54.7, 193.2)
- added U3: DRV8833, DRV8833:DRV8833, F.Cu at (211.4, 186.8)
- added U4: DRV8833, DRV8833:DRV8833, F.Cu at (231.2, 132.6)
- added U5: AMS1117, Package_TO_SOT_SMD:SOT-223-3_TabPin2, B.Cu at (244.7, 193.2)
- added W1: 5104, JUMPLER 5104:KEYSTONE_5104, B.Cu at (255.1, 127.5)
- added W2: 5104, JUMPLER 5104:KEYSTONE_5104, B.Cu at (65.1, 25.5)
- added W3: 5104, JUMPLER 5104:KEYSTONE_5104, B.Cu at (160.1, 25.5)
- added W4: 5104, JUMPLER 5104:KEYSTONE_5104, B.Cu at (255.1, 25.5)
- added W5: 5104, JUMPLER 5104:KEYSTONE_5104, B.Cu at (65.1, 127.5)
- added W6: 5104, JUMPLER 5104:KEYSTONE_5104, B.Cu at (160.1, 127.5)
- J11: value SWITCH -> BAT; footprint Connector_PinHeader_2.54mm:PinHeader_1x03_P2.54mm_Vertical -> TerminalBlock_Phoenix:TerminalBlock_Phoenix_MKDS-1,5-2_1x02_P5.00mm_Horizontal
- J12: value M1 -> SWITCH; footprint TerminalBlock_Phoenix:TerminalBlock_Phoenix_MKDS-1,5-2_1x02_P5.00mm_Horizontal -> Connector_PinHeader_2.54mm:PinHeader_1x03_P2.54mm_Vertical
- J13: value M2 -> M1
- J14: value SENSORES -> M2; footprint Connector_PinHeader_2.54mm:PinHeader_1x11_P2.54mm_Vertical -> TerminalBlock_Phoenix:TerminalBlock_Phoenix_MKDS-1,5-2_1x02_P5.00mm_Horizontal
- J15: value SWITCH -> SENSORES; footprint Connector_PinHeader_2.54mm:PinHeader_1x03_P2.54mm_Vertical -> Connector_PinHeader_2.54mm:PinHeader_1x11_P2.54mm_Vertical
- J16: value M1 -> BAT
- J17: value M2 -> SWITCH; footprint TerminalBlock_Phoenix:TerminalBlock_Phoenix_MKDS-1,5-2_1x02_P5.00mm_Horizontal -> Connector_PinHeader_2.54mm:PinHeader_1x03_P2.54mm_Vertical
- J18: value SENSORES -> M1; footprint Connector_PinHeader_2.54mm:PinHeader_1x11_P2.54mm_Vertical -> TerminalBlock_Phoenix:TerminalBlock_Phoenix_MKDS-1,5-2_1x02_P5.00mm_Horizontal
- J4: value BAT -> M1
- J5: value BAT -> M2
- R10, R19: value 0 -> 10k
- R12, R20: value 10k -> 220
- R13, R22: value 220 -> 0
- R15, R23: value 0 -> 1k
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Connections:
- J11 pad 2: Net-(J1-Pin_1) -> GND
- J12 pad 1: Net-(J4-Pin_1) -> Net-(J1-Pin_1)
- J12 pad 2: Net-(J4-Pin_2) -> Net-(J1-Pin_1)
- J13 pad 1: Net-(J5-Pin_1) -> Net-(J4-Pin_1)
- J13 pad 2: Net-(J5-Pin_2) -> Net-(J4-Pin_2)
- J14 pad 1: +3.3V -> Net-(J5-Pin_1)
- J14 pad 2: /S8 -> Net-(J5-Pin_2)
- J15 pad 1: Net-(J1-Pin_1) -> +3.3V
- J15 pad 2: Net-(J1-Pin_1) -> /S8
- J15 pad 3: Net-(D3-A) -> /S7
- J16 pad 1: Net-(J4-Pin_1) -> Net-(J1-Pin_1)
- J16 pad 2: Net-(J4-Pin_2) -> GND
- J17 pad 1: Net-(J5-Pin_1) -> Net-(J1-Pin_1)
- J17 pad 2: Net-(J5-Pin_2) -> Net-(J1-Pin_1)
- J18 pad 1: +3.3V -> Net-(J4-Pin_1)
- J18 pad 2: /S8 -> Net-(J4-Pin_2)
- J4 pad 1: Net-(J1-Pin_1) -> Net-(J4-Pin_1)
- J4 pad 2: GND -> Net-(J4-Pin_2)
- J5 pad 1: Net-(J1-Pin_1) -> Net-(J5-Pin_1)
- J5 pad 2: GND -> Net-(J5-Pin_2)
- R10 pad 1: GND -> Net-(C3-Pad1)
- R11 pad 1: Net-(C3-Pad1) -> Net-(C4-Pad1)
- R12 pad 1: Net-(C4-Pad1) -> Net-(D1-K)
- R13 pad 1: Net-(D1-K) -> /IN_M1_A
- R13 pad 2: GND -> Net-(U3-IN2)
- R14 pad 1: /IN_M1_A -> /IN_M2_B
- R14 pad 2: Net-(U3-IN2) -> Net-(U4-IN3)
- R15 pad 1: /IN_M2_B -> /BUZZER
- R15 pad 2: Net-(U4-IN3) -> Net-(Q1-B)
- R16 pad 1: /BUZZER -> Net-(C4-Pad1)
- R16 pad 2: Net-(Q1-B) -> /SW2
- R17 pad 1: Net-(C4-Pad1) -> Net-(C3-Pad1)
- R17 pad 2: /SW2 -> /SW1
- R18 pad 2: /SW1 -> GND
- R19 pad 1: GND -> Net-(C4-Pad1)
- R20 pad 1: Net-(C3-Pad1) -> Net-(D1-K)
- R21 pad 1: Net-(C4-Pad1) -> /IN_M1_A
- R21 pad 2: GND -> Net-(U3-IN2)
- R22 pad 1: Net-(D1-K) -> /IN_M2_B
- R22 pad 2: GND -> Net-(U4-IN3)
- R23 pad 1: /IN_M1_A -> /BUZZER
- R23 pad 2: Net-(U3-IN2) -> Net-(Q1-B)
- R24 pad 1: /IN_M2_B -> Net-(C4-Pad1)
- R24 pad 2: Net-(U4-IN3) -> /SW2
- R25 pad 1: /BUZZER -> Net-(C3-Pad1)
- R25 pad 2: Net-(Q1-B) -> /SW1
- R26 pad 1: Net-(C4-Pad1) -> Net-(C3-Pad1)
- R26 pad 2: /SW2 -> GND
- R27 pad 1: Net-(C3-Pad1) -> Net-(C4-Pad1)
- R27 pad 2: /SW1 -> GND
- R28 pad 1: GND -> Net-(D1-K)
- R29 pad 1: Net-(C3-Pad1) -> /IN_M1_A
- R29 pad 2: GND -> Net-(U3-IN2)
- R30 pad 1: Net-(C4-Pad1) -> /IN_M2_B
- R30 pad 2: GND -> Net-(U4-IN3)
- R31 pad 1: Net-(D1-K) -> /BUZZER
- R31 pad 2: GND -> Net-(Q1-B)
- R32 pad 1: /IN_M1_A -> Net-(C4-Pad1)
- R32 pad 2: Net-(U3-IN2) -> /SW2
- R33 pad 1: /IN_M2_B -> Net-(C3-Pad1)
- R33 pad 2: Net-(U4-IN3) -> /SW1
- R34 pad 1: /BUZZER -> Net-(C3-Pad1)
- R34 pad 2: Net-(Q1-B) -> GND
- R35 pad 2: /SW2 -> GND
- R36 pad 1: Net-(C3-Pad1) -> Net-(D1-K)
- R36 pad 2: /SW1 -> GND
- R46 pad 1: GND -> /IN_M2_B
- R46 pad 2: GND -> Net-(U4-IN3)
- R47 pad 1: Net-(C3-Pad1) -> /BUZZER
- R47 pad 2: GND -> Net-(Q1-B)
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Routing:
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Other:
- board size 246 x 195 mm -> 252 x 197 mm
- board text added: "* MotorBoard FIE * A: Sanchez Samuel * V1.4 - 2025"
- board text added: "2025 - V1.4"
- board text removed: "* MotorBoard FIE * A: Sanchez Samuel * V1.3 - 2025"
- board text removed: "2025 - V1.3"
